File: board1-pdb/board1-pdb.kicad_pcb (KiCad board)
At the start: 2 copper layers, 51 x 54 mm, 32 parts, among them J1 XT60PW-M, J2 SM04B-SRSS-TB, J3 XT60PW-F, J4 XT60PW-F, J5 XT60PW-F, J6 XT60PW-F, U1 ACS773LCB-100B-PFF, U2 LMR33630ADDA, U3 AMS1117-3.3

Commit message: chore: Moved to board1-pdb project
Other:
- board text added: "H. Juarez FC-PDB-001-A 2026"
Changed lines of the file:
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@@
   (gr_rect (start 114 79) (end 165 133)
     (stroke (width 0.05) (type default)) (fill none) (layer "Edge.Cuts"))
+  (gr_text "H. Juarez\nFC-PDB-001-A\n2026" (at 144.272 84.836) (layer "F.SilkS")
+    (effects (font (size 1 1) (thickness 0.15)) (justify left bottom))
+  )
   (segment (start 144.424 89.662) (end 145.424 89.662) (width 0.5) (layer "F.Cu") (net 1))
   (segment (start 144.121 89.359) (end 144.424 89.662) (width 0.5) (layer "F.Cu") (net 1))
